File: Game_Cat_R3_BUTTONS.kicad_sch (KiCad schematic)
At the start: 67 parts, among them J1 Joystick, J2 UART, J3 PWM, J4 CAN, Q1 MMBT3906, Q2 MMBT3904, Q3 BSS138, Q4 BSS138, Q5 BSS138, Q6 BSS138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

Commit message: 26/12/13/A
Other:
- note added: "CAN BUS"
Changed lines of the file:
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@@
     (effects (font (size 2.032 2.032) (thickness 0.4064) bold) (justify left bottom))
   )
-  (text "BUZZER PWM" (at 170.18 97.155 0)
+  (text "CAN BUS" (at 170.18 97.155 0)
     (effects (font (size 2.032 2.032) (thickness 0.4064) bold) (justify left bottom))
   )
